File: ESP_PD210.kicad_pcb (KiCad board)
At the start: 4 copper layers, 88.8 x 13 mm, 66 parts, among them J1 TTL, J2 CART, J3 USB_C_Receptacle_USB2.0, Q1 NPN, Q2 SE30P09D, SW1 Rocker, SW2 Move, U1 SSD1316, U2 ESP8684, U3 AD8628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

Commit message: Replace the OPA with OPA188
Parts:
- U3: value AD8628 -> OPA188
Routing:
- net GND: track 7.58 -> 3.41 mm, vias 23 -> 24
- added copper zone on In2.Cu, net GND
Changed lines of the file:
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@@
       (effects (font (size 1 1) (thickness 0.15)) (justify mirror))
     )
-    (fp_text value "AD8628" (at 0 -2.4) (layer "B.Fab")
+    (fp_text value "OPA188" (at 0 -2.4) (layer "B.Fab")
       (effects (font (size 1 1) (thickness 0.15)) (justify mirror))
     )
@@
     (pts (xy 188.63 92.56) (xy 188.63 105.56))
     (height -4.76069)
-    (gr_text "511.8110 mils" (at 192.24069 99.06 90) (layer "User.1")
+    (gr_text "13.0000 mm" (at 192.24069 99.06 90) (layer "User.1")
       (effects (font (size 1 1) (thickness 0.15)))
     )
@@
     (pts (xy 99.78 92.18) (xy 188.63 92.19))
     (height -2.96)
-    (gr_text "3498.0315 mils" (at 144.205462 88.075 359.9935514) (layer "User.1")
+    (gr_text "88.8500 mm" (at 144.205462 88.075 359.9935514) (layer "User.1")
       (effects (font (size 1 1) (thickness 0.15)))
     )
@@
   (via (at 160.828002 98.303012) (size 0.6048) (drill 0.3) (layers "F.Cu" "B.Cu") (net 1))
   (via (at 179.25 94.95) (size 0.6048) (drill 0.3) (layers "F.Cu" "B.Cu") (remove_unused_layers) (keep_end_layers) (net 1))
+  (via (at 152.489992 100.419992) (size 0.6048) (drill 0.3) (layers "F.Cu" "B.Cu") (free) (net 1))
   (via (at 173.34 104.01) (size 0.6048) (drill 0.3) (layers "F.Cu" "B.Cu") (remove_unused_layers) (keep_end_layers) (net 1))
   (via (at 160.828002 99.065012) (size 0.6048) (drill 0.3) (layers "F.Cu" "B.Cu") (net 1))
@@
   (via (at 162.352002 99.827012) (size 0.6048) (drill 0.3) (layers "F.Cu" "B.Cu") (net 1))
   (via (at 156.51 97.97) (size 0.6048) (drill 0.3) (layers "F.Cu" "B.Cu") (free) (net 1))
-  (segment (start 178.780001 95.65) (end 178.780001 95.419999) (width 0.381) (layer "B.Cu") (net 1))
-  (segment (start 178.780001 95.419999) (end 179.25 94.95) (width 0.381) (layer "B.Cu") (net 1))
-  (segment (start 185.6092 95.4866) (end 186.3508 94.745) (width 0.254) (layer "B.Cu") (net 1))
-  (segment (start 185.6092 96.578036) (end 185.6092 95.4866) (width 0.254) (layer "B.Cu") (net 1))
-  (segment (start 186.7475 99.758036) (end 185.61 99.758036) (width 0.254) (layer "B.Cu") (net 1))
   (segment (start 175.6 103.68) (end 175 103.68) (width 0.254) (layer "F.Cu") (net 2))
   (segment (start 173.905 102.585) (end 171.26 102.585) (width 0.254) (layer "F.Cu") (net 2))
@@
   (via (at 166.540002 96.925511) (size 0.6048) (drill 0.3) (layers "F.Cu" "B.Cu") (remove_unused_layers) (keep_end_layers) (net 6))
   (via (at 168.429991 95.375) (size 0.6048) (drill 0.3) (layers "F.Cu" "B.Cu") (remove_unused_layers) (keep_end_layers) (free) (net 6))
-  (segment (start 138.02901 102.7982) (end 148.4118 102.7982) (width 0.254) (layer "In2.Cu") (net 6))
+  (segment (start 148.4118 102.7982) (end 154.43 96.78) (width 0.254) (layer "In2.Cu") (net 6))
   (segment (start 158.090012 96.78) (end 158.250001 96.939989) (width 0.254) (layer "In2.Cu") (net 6))
   (segment (start 166.538709 96.926804) (end 166.540002 96.925511) (width 0.254) (layer "In2.Cu") (net 6))
+  (segment (start 166.87948 96.925511) (end 168.429991 95.375) (width 0.254) (layer "In2.Cu") (net 6))
   (segment (start 154.43 96.78) (end 158.090012 96.78) (width 0.254) (layer "In2.Cu") (net 6))
-  (segment (start 166.87948 96.925511) (end 168.429991 95.375) (width 0.254) (layer "In2.Cu") (net 6))
-  (segment (start 137.827213 102.999997) (end 138.02901 102.7982) (width 0.254) (layer "In2.Cu") (net 6))
+  (segment (start 136.230004 102.999997) (end 136.431801 102.7982) (width 0.254) (layer "In2.Cu") (net 6))
   (segment (start 163.73 103.96) (end 163.52 103.96) (width 0.254) (layer "In2.Cu") (net 6))
-  (segment (start 136.230004 102.999997) (end 137.827213 102.999997) (width 0.254) (layer "In2.Cu") (net 6))
   (segment (start 165.4 102.29) (end 163.73 103.96) (width 0.254) (layer "In2.Cu") (net 6))
   (segment (start 167.92 98.305509) (end 167.92 99.24) (width 0.254) (layer "In2.Cu") (net 6))
   (segment (start 166.540002 96.925511) (end 167.92 98.305509) (width 0.254) (layer "In2.Cu") (net 6))
   (segment (start 166.540002 96.925511) (end 166.87948 96.925511) (width 0.254) (layer "In2.Cu") (net 6))
-  (segment (start 148.4118 102.7982) (end 154.43 96.78) (width 0.254) (layer "In2.Cu") (net 6))
+  (segment (start 136.431801 102.7982) (end 148.4118 102.7982) (width 0.254) (layer "In2.Cu") (net 6))
   (segment (start 175.900001 101.38) (end 176.120001 101.6) (width 0.381) (layer "B.Cu") (net 6))
   (segment (start 136.230007 103) (end 136.230004 102.999997) (width 0.254) (layer "B.Cu") (net 6))
@@
   (segment (start 163.5525 99.315) (end 165.151854 99.315) (width 0.1524) (layer "F.Cu") (net 34))
   (via (at 165.28001 99.849991) (size 0.6048) (drill 0.3) (layers "F.Cu" "B.Cu") (remove_unused_layers) (keep_end_layers) (net 34))
-  (segment (start 165.28 99.85) (end 169.83 99.85) (width 0.1524) (layer "B.Cu") (net 34))
-  (segment (start 169.83 99.85) (end 171.79 97.89) (width 0.1524) (layer "B.Cu") (net 34))
+  (segment (start 168.060948 99.85) (end 170.020948 97.89) (width 0.1524) (layer "B.Cu") (net 34))
+  (segment (start 165.28 99.85) (end 168.060948 99.85) (width 0.1524) (layer "B.Cu") (net 34))
+  (segment (start 170.020948 97.89) (end 171.79 97.89) (width 0.1524) (layer "B.Cu") (net 34))
   (segment (start 143.855 95.935) (end 144.49 96.57) (width 0.254) (layer "B.Cu") (net 35))
   (segment (start 143.59 97.47) (end 144.49 96.57) (width 0.254) (layer "B.Cu") (net 35))
@@
   (segment (start 164.45 102.79) (end 164.45 103.525) (width 0.254) (layer "F.Cu") (net 37))
   (segment (start 162.73 102.24) (end 163.9 102.24) (width 0.254) (layer "F.Cu") (net 37))
+  (segment (start 144.7252 96.6352) (end 143.871852 95.781852) (width 0.1524) (layer "F.Cu") (net 38))
+  (segment (start 149.5843 97.72) (end 148.46 97.72) (width 0.1524) (layer "F.Cu") (net 38))
   (segment (start 160.071636 96.46) (end 160.07 96.46) (width 0.1524) (layer "F.Cu") (net 38))
   (segment (start 160.34 96.728364) (end 160.071636 96.46) (width 0.1524) (layer "F.Cu") (net 38))
+  (segment (start 160.07 96.46) (end 159.51 95.9) (width 0.1524) (layer "F.Cu") (net 38))
   (segment (start 149.81 97.4943) (end 149.5843 97.72) (width 0.1524) (layer "F.Cu") (net 38))
+  (segment (start 159.51 95.9) (end 159.51 95.1399) (width 0.1524) (layer "F.Cu") (net 38))
   (segment (start 148.46 97.72) (end 147.3752 96.6352) (width 0.1524) (layer "F.Cu") (net 38))
-  (segment (start 149.5843 97.72) (end 148.46 97.72) (width 0.1524) (layer "F.Cu") (net 38))
-  (segment (start 160.07 96.46) (end 159.51 95.9) (width 0.1524) (layer "F.Cu") (net 38))
-  (segment (start 159.51 95.9) (end 159.51 95.1399) (width 0.1524) (layer "F.Cu") (net 38))
+  (segment (start 160.34 97.1025) (end 160.34 96.728364) (width 0.1524) (layer "F.Cu") (net 38))
   (segment (start 147.3752 96.6352) (end 144.7252 96.6352) (width 0.1524) (layer "F.Cu") (net 38))
-  (segment (start 160.34 97.1025) (end 160.34 96.728364) (width 0.1524) (layer "F.Cu") (net 38))
-  (segment (start 144.7252 96.6352) (end 143.871852 95.781852) (width 0.1524) (layer "F.Cu") (net 38))
   (via (at 159.509993 95.139891) (size 0.6048) (drill 0.3) (layers "F.Cu" "B.Cu") (remove_unused_layers) (keep_end_layers) (net 38))
   (via (at 149.81 97.4943) (size 0.6048) (drill 0.3) (layers "F.Cu" "B.Cu") (remove_unused_layers) (keep_end_layers) (net 38))
@@
   (segment (start 164.885 97.815) (end 166.305 96.395) (width 0.1524) (layer "F.Cu") (net 44))
   (segment (start 169.875 96.395) (end 170.305 96.825) (width 0.254) (layer "F.Cu") (net 44))
-  (segment (start 157.99 101.2) (end 160.1675 101.2) (width 0.381) (layer "F.Cu") (net 45))
+  (segment (start 157.990007 101.200001) (end 160.269098 101.200001) (width 0.381) (layer "F.Cu") (net 45))
   (segment (start 157.035 101.2) (end 157.99 101.2) (width 0.381) (layer "F.Cu") (net 45))
-  (segment (start 160.167498 101.200001) (end 160.339989 101.027509) (width 0.254) (layer "F.Cu") (net 45))
   (segment (start 175.900001 96.07) (end 175.900001 95.65) (width 0.381) (layer "B.Cu") (net 49))
   (segment (start 176.340001 97.0625) (end 176.340001 96.51) (width 0.381) (layer "B.Cu") (net 49))
@@
     (min_thickness 0.254)
     (keepout (tracks allowed) (vias allowed) (pads allowed ) (copperpour not_allowed) (footprints allowed))
-    (fill (thermal_gap 0.508) (thermal_bridge_width 0.508) (smoothing fillet) (radius 0.508))
+    (fill (thermal_gap 0.508) (thermal_bridge_width 0.508))
     (polygon
       (pts
-        (xy 163.54 101.01)
-        (xy 159.62 101.01)
-        (xy 159.62 97.08)
-        (xy 163.54 97.08)
+        (xy 163.6416 101.11486)
+        (xy 159.54126 101.11486)
+        (xy 159.54126 97.01468)
+        (xy 163.6416 97.01468)
       )
     )
@@
     (connect_pads yes (clearance 0))
     (min_thickness 0.254) (filled_areas_thickness no)
-    (fill yes (thermal_gap 0.508) (thermal_bridge_width 0.508) (smoothing fillet) (radius 0.508))
+    (fill yes (thermal_gap 0.508) (thermal_bridge_width 0.508))
     (polygon
       (pts
@@
       )
     )
+  )
+  (zone (net 1) (net_name "GND") (layer "In2.Cu") (hatch edge 0.508)
+    (connect_pads (clearance 0))
+    (min_thickness 0.254) (filled_areas_thickness no)
+    (fill yes (thermal_gap 0.508) (thermal_bridge_width 0.508))
+    (polygon
+      (pts
+        (xy 158.310135 102.70004)
+        (xy 151.419999 102.709952)
+        (xy 151.420217 99.559363)
+        (xy 158.310353 99.562111)
+      )
+    )

Commit message: 优化电源走线，增加 adc 处滤波电容
Parts:
- added C24: 0.1uF, Capacitor_SMD:C_0402_1005Metric, B.Cu at (135.0, 103.5)
- added C25: 0.1uF, Capacitor_SMD:C_0402_1005Metric, B.Cu at (161.2, 103.3)
- R10: value 1.2M -> 390K
- R9: value 1K -> 390
Routing:
- net +3V3: track 81.5 -> 75.3 mm, vias 10 -> 11
- net /TEMP: track 26.1 -> 27.0 mm
- net Net-(D1-Pad2): track 8.30 -> 7.66 mm
- added copper zone on B.Cu, net +3V3
- added copper zone on F.Cu, net +3V3

Commit message: Optimize the layout
Parts:
- moved AE1 8.84 mm to (160.9, 110.0)
- moved C10 8.84 mm to (173.5, 108.0)
- moved C11 8.84 mm to (169.4, 109.5)
- moved C14 8.84 mm to (141.0, 109.5)
- moved C15 8.84 mm to (171.2, 101.5)
- moved C16 8.84 mm to (173.4, 106.4)
- moved C19 8.84 mm to (192.4, 102.7)
- moved C22 8.84 mm to (161.9, 106.4)
- moved C24 8.84 mm to (141.8, 109.1)
- moved C25 8.84 mm to (167.9, 109.0)
- moved C4 8.84 mm to (163.9, 105.3)
- moved C5 8.84 mm to (164.5, 103.4)
- moved C6 8.84 mm to (162.4, 102.0)
- moved L2 8.84 mm to (162.4, 103.8)
- moved L3 8.84 mm to (184.7, 107.3)
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Routing:
- net +3V3: track 75.3 -> 43.1 mm
- net GND: vias 24 -> 23
- removed copper zone on In2.Cu, net GND
